Commit message: djakd

File: rover_description/urdf/diff_drive.xacro (robot description, xacro)
@@ -19,5 +19,5 @@
         <!-- TF correcto -->
         <frame_id>odom</frame_id>
-        <child_frame_id>base_link</child_frame_id>
+        <child_frame_id>base_footprint</child_frame_id>
         <publish_odom>false</publish_odom>
         <publish_odom_tf>false</publish_odom_tf>

File: rover_description/urdf/rover.xacro (robot description, xacro)
@@ -16,7 +16,11 @@
     <color rgba="0.5 0.5 0.5 1"/>
   </material>
-  <!-- ===================== -->
-  <!-- BASE -->
-  <!-- ===================== -->
+  <!-- BASES -->
+  <link name="base_footprint"/>
+  <joint name="base_link_joint" type="fixed">
+    <parent link="base_footprint"/>
+    <child link="base_link"/>
+    <origin xyz="0 0 0" rpy="0 0 0"/>
+  </joint>
   <link name="base_link">
     <visual>
