Commit message: prueba

File: rover_description/urdf/lidar.xacro (robot description, xacro)
@@ -2,23 +2,46 @@
 <robot xmlns:xacro="http://www.ros.org/wiki/xacro">
   <xacro:macro name="lidar_plugin" params="prefix">
-    <gazebo reference="laser_link">
-      <sensor type="ray" name="lidar">
+    <xacro:property name="lidar_height" value="0.4"/>
+    <xacro:property name="lidar_radius" value="0.05"/>
+    <link name="lidar_link">
+      <visual>
+        <geometry>
+          <cylinder radius="${lidar_radius}" length="0.05"/>
+        </geometry>
+        <material name="black"/>
+      </visual>
+      <inertial>
+        <mass value="0.5"/>
+        <origin xyz="0 0 0"/>
+        <inertia ixx="0.001" ixy="0" ixz="0"
+                 iyy="0.001" iyz="0" izz="0.001"/>
+      </inertial>
+    </link>
+    <joint name="lidar_joint" type="fixed">
+      <parent link="base_link"/>
+      <child link="lidar_link"/>
+      <origin xyz="0 0 ${lidar_height}" rpy="0 0 3.14159"/>
+    </joint>
+    <gazebo reference="lidar_link">
+      <sensor name="lidar_sensor" type="gpu_lidar">
+        <gz_frame_id>${prefix}/lidar_link</gz_frame_id>
         <update_rate>10</update_rate>
+        <topic>/model/${prefix}/scan</topic>
         <ray>
           <scan>
             <horizontal>
-              <samples>360</samples>
-              <min_angle>-3.14</min_angle>
-              <max_angle>3.14</max_angle>
+              <samples>720</samples>
+              <resolution>1</resolution>
+              <min_angle>-3.1416</min_angle>
+              <max_angle>3.1416</max_angle>
             </horizontal>
           </scan>
           <range>
-            <min>0.1</min>
+            <min>0.12</min>
             <max>10.0</max>
+            <resolution>0.01</resolution>
           </range>
         </ray>
-        <always_on>true</always_on>
         <visualize>true</visualize>
-        <topic>/model/rover/scan</topic>
       </sensor>
     </gazebo>

Commit message: el arbol de transformacion esta bien pero en rviz parpadea

File: rover_description/urdf/lidar.xacro (robot description, xacro)
@@ -4,5 +4,5 @@
     <xacro:property name="lidar_height" value="0.4"/>
     <xacro:property name="lidar_radius" value="0.05"/>
-    <link name="lidar_link">
+    <link name="$(arg prefix)lidar_link">
       <visual>
         <geometry>
@@ -18,14 +18,14 @@
       </inertial>
     </link>
-    <joint name="lidar_joint" type="fixed">
-      <parent link="base_link"/>
-      <child link="lidar_link"/>
+    <joint name="$(arg prefix)lidar_joint" type="fixed">
+      <parent link="$(arg prefix)base_link"/>
+      <child link="$(arg prefix)lidar_link"/>
       <origin xyz="0 0 ${lidar_height}" rpy="0 0 3.14159"/>
     </joint>
-    <gazebo reference="lidar_link">
-      <sensor name="lidar_sensor" type="gpu_lidar">
-        <gz_frame_id>${prefix}/lidar_link</gz_frame_id>
+    <gazebo reference="$(arg prefix)lidar_link">
+      <sensor name="$(arg prefix)lidar_sensor" type="gpu_lidar">
+        <gz_frame_id>$(arg prefix)lidar_link</gz_frame_id>
         <update_rate>10</update_rate>
-        <topic>/model/${prefix}/scan</topic>
+        <topic>$(arg prefix)scan</topic>
         <ray>
           <scan>

File: rover_description/urdf/rover.xacro (robot description, xacro)
@@ -1,6 +1,19 @@
 <?xml version="1.0"?>
-<robot name="rover" xmlns:xacro="http://www.ros.org/wiki/xacro">
-  <xacro:include filename="diff_drive.xacro"/>
-  <xacro:include filename="lidar.xacro"/>
+<robot xmlns:xacro="http://www.ros.org/wiki/xacro">
+  <!-- Macro para inercia de cajas -->
+  <xacro:macro name="box_inertia" params="m x y z o_xyz o_rpy">
+    <inertial>
+      <mass value="${m}"/>
+      <origin xyz="${o_xyz}" rpy="${o_rpy}"/>
+      <inertia
+        ixx="${m/12.0*(y*y + z*z)}"
+        ixy="0"
+        ixz="0"
+        iyy="${m/12.0*(x*x + z*z)}"
+        iyz="0"
+        izz="${m/12.0*(x*x + y*y)}"
+      />
+    </inertial>
+  </xacro:macro>
   <!-- Parámetros -->
   <xacro:property name="wheel_radius" value="0.15"/>
@@ -17,11 +30,11 @@
   </material>
   <!-- BASES -->
-  <link name="base_footprint"/>
-  <joint name="base_link_joint" type="fixed">
-    <parent link="base_footprint"/>
-    <child link="base_link"/>
+  <link name="$(arg prefix)base_footprint"/>
+  <joint name="$(arg prefix)base_link_joint" type="fixed">
+    <parent link="$(arg prefix)base_footprint"/>
+    <child link="$(arg prefix)base_link"/>
     <origin xyz="0 0 0" rpy="0 0 0"/>
   </joint>
-  <link name="base_link">
+  <link name="$(arg prefix)base_link">
     <visual>
       <origin xyz="0 0 0.175" rpy="0 0 0"/>
@@ -46,5 +59,5 @@
   <!-- RUEDAS -->
   <!-- ===================== -->
-  <link name="left_front_wheel">
+  <link name="$(arg prefix)left_front_wheel">
     <visual>
       <geometry>
@@ -65,5 +78,5 @@
     </inertial>
   </link>
-  <link name="right_front_wheel">
+  <link name="$(arg prefix)right_front_wheel">
     <visual>
       <geometry>
@@ -84,5 +97,5 @@
     </inertial>
   </link>
-  <link name="left_rear_wheel">
+  <link name="$(arg prefix)left_rear_wheel">
     <visual>
       <geometry>
@@ -103,5 +116,5 @@
     </inertial>
   </link>
-  <link name="right_rear_wheel">
+  <link name="$(arg prefix)right_rear_wheel">
     <visual>
       <geometry>
@@ -122,45 +135,27 @@
     </inertial>
   </link>
-  <joint name="left_front_wheel_joint" type="continuous">
-    <parent link="base_link"/>
-    <child link="left_front_wheel"/>
+  <joint name="$(arg prefix)left_front_wheel_joint" type="continuous">
+    <parent link="$(arg prefix)base_link"/>
+    <child link="$(arg prefix)left_front_wheel"/>
     <origin xyz="0.3 ${wheel_separation} 0.15" rpy="1.57 0 0"/>
     <axis xyz="0 0 1"/>
   </joint>
-  <joint name="right_front_wheel_joint" type="continuous">
-    <parent link="base_link"/>
-    <child link="right_front_wheel"/>
+  <joint name="$(arg prefix)right_front_wheel_joint" type="continuous">
+    <parent link="$(arg prefix)base_link"/>
+    <child link="$(arg prefix)right_front_wheel"/>
     <origin xyz="0.3 -${wheel_separation} 0.15" rpy="1.57 0 0"/>
     <axis xyz="0 0 1"/>
   </joint>
-  <joint name="left_rear_wheel_joint" type="continuous">
-    <parent link="base_link"/>
-    <child link="left_rear_wheel"/>
+  <joint name="$(arg prefix)left_rear_wheel_joint" type="continuous">
+    <parent link="$(arg prefix)base_link"/>
+    <child link="$(arg prefix)left_rear_wheel"/>
     <origin xyz="-0.3 ${wheel_separation} 0.15" rpy="1.57 0 0"/>
     <axis xyz="0 0 1"/>
   </joint>
-  <joint name="right_rear_wheel_joint" type="continuous">
-    <parent link="base_link"/>
-    <child link="right_rear_wheel"/>
+  <joint name="$(arg prefix)right_rear_wheel_joint" type="continuous">
+    <parent link="$(arg prefix)base_link"/>
+    <child link="$(arg prefix)right_rear_wheel"/>
     <origin xyz="-0.3 -${wheel_separation} 0.15" rpy="1.57 0 0"/>
     <axis xyz="0 0 1"/>
   </joint>
-  <!-- ===================== -->
-  <!-- LIDAR -->
-  <!-- ===================== -->
-  <link name="laser_link">
-    <visual>
-      <geometry>
-        <cylinder radius="0.05" length="0.05"/>
-      </geometry>
-      <material name="gray"/>
-    </visual>
-  </link>
-  <joint name="laser_joint" type="fixed">
-    <parent link="base_link"/>
-    <child link="laser_link"/>
-    <origin xyz="0.3 0 0.4"/>
-  </joint>
-  <xacro:simulacion prefix="rover"/>
-  <xacro:lidar_plugin prefix="rover"/>
 </robot>
