Commit message: rover con lidar y camara, he añadido un fichero para probar que evite obstaculos y otro en el que mezclo evitar obstaculos con seguir los puntos del dron

File: rover_description/urdf/gazebo_plugins.xacro (robot description, xacro)
@@ -10,5 +10,5 @@
       <right_joint>$(arg prefix)right_front_wheel_joint</right_joint>
       <right_joint>$(arg prefix)right_rear_wheel_joint</right_joint>
-      <wheel_separation>0.41</wheel_separation>
+      <wheel_separation>0.9</wheel_separation>
       <wheel_radius>0.15</wheel_radius>
       <!--Topic para la odometría-->

File: rover_description/urdf/lidar.xacro (robot description, xacro)
@@ -1,49 +1,46 @@
 <?xml version="1.0"?>
 <robot xmlns:xacro="http://www.ros.org/wiki/xacro">
-  <xacro:macro name="lidar_plugin" params="prefix">
-    <xacro:property name="lidar_height" value="0.4"/>
-    <xacro:property name="lidar_radius" value="0.05"/>
-    <link name="$(arg prefix)lidar_link">
-      <visual>
-        <geometry>
-          <cylinder radius="${lidar_radius}" length="0.05"/>
-        </geometry>
-        <material name="black"/>
-      </visual>
-      <inertial>
-        <mass value="0.5"/>
-        <origin xyz="0 0 0"/>
-        <inertia ixx="0.001" ixy="0" ixz="0"
-                 iyy="0.001" iyz="0" izz="0.001"/>
-      </inertial>
-    </link>
-    <joint name="$(arg prefix)lidar_joint" type="fixed">
-      <parent link="$(arg prefix)base_link"/>
-      <child link="$(arg prefix)lidar_link"/>
-      <origin xyz="0 0 ${lidar_height}" rpy="0 0 3.14159"/>
-    </joint>
-    <gazebo reference="$(arg prefix)lidar_link">
-      <sensor name="$(arg prefix)lidar_sensor" type="gpu_lidar">
-        <gz_frame_id>$(arg prefix)lidar_link</gz_frame_id>
-        <update_rate>10</update_rate>
-        <topic>$(arg prefix)scan</topic>
-        <ray>
-          <scan>
-            <horizontal>
-              <samples>720</samples>
-              <resolution>1</resolution>
-              <min_angle>-3.1416</min_angle>
-              <max_angle>3.1416</max_angle>
-            </horizontal>
-          </scan>
-          <range>
-            <min>0.12</min>
-            <max>10.0</max>
-            <resolution>0.01</resolution>
-          </range>
-        </ray>
-        <visualize>true</visualize>
-      </sensor>
-    </gazebo>
-  </xacro:macro>
+  <xacro:property name="lidar_radius" value="0.05"/>
+  <xacro:property name="lidar_length" value="0.04"/>
+      <joint name="$(arg prefix)laser_joint" type="fixed"> <parent link="$(arg prefix)base_link"/>
+        <child link="$(arg prefix)lidar_link"/> <origin xyz="0 0 0.45" rpy="0 0 0"/>
+      </joint>
+      <link name="$(arg prefix)lidar_link">
+        <visual>
+          <origin xyz="0 0 0" rpy="0 0 0"/>
+          <geometry>
+            <cylinder radius="${lidar_radius}" length="${lidar_length}"/>
+          </geometry>
+          <material name="white"/>
+        </visual>
+        <collision>
+          <origin xyz="0 0 0" rpy="0 0 0"/>
+          <geometry>
+            <cylinder radius="${lidar_radius}" length="${lidar_length}"/>
+          </geometry>
+        </collision>
+      </link>
+      <gazebo reference="$(arg prefix)lidar_link">
+        <sensor name="lidar_sensor" type="gpu_lidar">
+          <gz_frame_id>$(arg prefix)lidar_link</gz_frame_id>
+          <update_rate>10</update_rate>
+          <topic>$(arg prefix)scan</topic>
+          <ray>
+            <scan>
+              <horizontal>
+                <samples>720</samples>
+                <resolution>1</resolution>
+                <min_angle>-3.1416</min_angle>
+                <max_angle>3.1416</max_angle>
+              </horizontal>
+            </scan>
+            <range>
+              <min>0.12</min>
+              <max>10.0</max>
+              <resolution>0.01</resolution>
+            </range>
+          </ray>
+          <visualize>true</visualize>
+        </sensor>
+      </gazebo>
 </robot>

File: rover_description/urdf/robot.urdf.xacro (robot description, xacro)
@@ -5,3 +5,4 @@
     <xacro:include filename="gazebo_plugins.xacro"/>
     <xacro:include filename="lidar.xacro"/>
+    <xacro:include filename="camera.xacro"/>
 </robot>

File: rover_description/urdf/rover.xacro (robot description, xacro)
@@ -38,5 +38,5 @@
   <link name="$(arg prefix)base_link">
     <visual>
-      <origin xyz="0 0 0.175" rpy="0 0 0"/>
+      <origin xyz="0 0 0.25" rpy="0 0 0"/>
       <geometry>
         <box size="1 0.7 0.35"/>
@@ -44,5 +44,5 @@
     </visual>
     <collision>
-      <origin xyz="0 0 0.175"/>
+      <origin xyz="0 0 0.25"/>
       <geometry>
         <box size="1 0.7 0.35"/>
@@ -138,5 +138,5 @@
     <parent link="$(arg prefix)base_link"/>
     <child link="$(arg prefix)left_front_wheel"/>
-    <origin xyz="0.3 ${wheel_separation} 0.15" rpy="1.57 0 0"/>
+    <origin xyz="0.3 ${wheel_separation} 0.15" rpy="-1.57 0 0"/>
     <axis xyz="0 0 1"/>
   </joint>
@@ -144,5 +144,5 @@
     <parent link="$(arg prefix)base_link"/>
     <child link="$(arg prefix)right_front_wheel"/>
-    <origin xyz="0.3 -${wheel_separation} 0.15" rpy="1.57 0 0"/>
+    <origin xyz="0.3 -${wheel_separation} 0.15" rpy="-1.57 0 0"/>
     <axis xyz="0 0 1"/>
   </joint>
@@ -150,5 +150,5 @@
     <parent link="$(arg prefix)base_link"/>
     <child link="$(arg prefix)left_rear_wheel"/>
-    <origin xyz="-0.3 ${wheel_separation} 0.15" rpy="1.57 0 0"/>
+    <origin xyz="-0.3 ${wheel_separation} 0.15" rpy="-1.57 0 0"/>
     <axis xyz="0 0 1"/>
   </joint>
@@ -156,6 +156,30 @@
     <parent link="$(arg prefix)base_link"/>
     <child link="$(arg prefix)right_rear_wheel"/>
-    <origin xyz="-0.3 -${wheel_separation} 0.15" rpy="1.57 0 0"/>
+    <origin xyz="-0.3 -${wheel_separation} 0.15" rpy="-1.57 0 0"/>
     <axis xyz="0 0 1"/>
   </joint>
+  <gazebo reference="$(arg prefix)left_front_wheel">
+    <mu1>0.2</mu1>
+    <mu2>0.2</mu2>
+    <kp>1000000.0</kp>
+    <kd>1.0</kd>
+  </gazebo>
+  <gazebo reference="$(arg prefix)right_front_wheel">
+    <mu1>0.2</mu1>
+    <mu2>0.2</mu2>
+    <kp>1000000.0</kp>
+    <kd>1.0</kd>
+  </gazebo>
+  <gazebo reference="$(arg prefix)left_rear_wheel">
+    <mu1>0.2</mu1>
+    <mu2>0.2</mu2>
+    <kp>1000000.0</kp>
+    <kd>1.0</kd>
+  </gazebo>
+  <gazebo reference="$(arg prefix)right_rear_wheel">
+    <mu1>0.2</mu1>
+    <mu2>0.2</mu2>
+    <kp>1000000.0</kp>
+    <kd>1.0</kd>
+  </gazebo>
 </robot>
