Commit message: Arreglado posicion lidar y abb

File: multi_robot_bringup/urdf/rover_abb.xacro (robot description, xacro)
@@ -10,5 +10,5 @@
         <parent link="$(arg prefix)base_link"/>
         <child link="arm_base_link"/>
-        <origin xyz="0.2 0 0.352" rpy="0 0 0"/>
+        <origin xyz="0 0 0.352" rpy="0 0 0"/>
     </joint>
 </robot>

File: rover_description/urdf/lidar.xacro (robot description, xacro)
@@ -4,5 +4,5 @@
   <xacro:property name="lidar_length" value="0.04"/>
       <joint name="$(arg prefix)laser_joint" type="fixed"> <parent link="$(arg prefix)base_link"/>
-        <child link="$(arg prefix)lidar_link"/> <origin xyz="0 0 0.45" rpy="0 0 0"/>
+        <child link="$(arg prefix)lidar_link"/> <origin xyz="0.25 0 0.45" rpy="0 0 0"/>
       </joint>
       <link name="$(arg prefix)lidar_link">

Commit message: fix: ajustar altura y visibilidad del brazo ABB en Gazebo

File: multi_robot_bringup/urdf/rover_abb.xacro (robot description, xacro)
@@ -10,5 +10,5 @@
         <parent link="$(arg prefix)base_link"/>
         <child link="arm_base_link"/>
-        <origin xyz="0 0 0.352" rpy="0 0 0"/>
+        <origin xyz="0 0 0.425" rpy="0 0 0"/>
     </joint>
 </robot>
