Commit message: Movimiento en gazebo

File: abb_irb120_description/urdf/irb120_3_58_macro.xacro (robot description, xacro)
@@ -1,4 +1,6 @@
 <?xml version="1.0"?>
 <robot name="irb120_3_58" xmlns:xacro="http://www.ros.org/wiki/xacro">
+  <material name="light_grey"><color rgba="0.9 0.9 0.9 1"/></material>
+  <material name="grey"><color rgba="0.4 0.4 0.4 1"/></material>
   <xacro:macro name="abb_irb120_3_58" params="prefix">
     <!-- link list -->
@@ -14,4 +16,5 @@
           <mesh filename="package://abb_irb120_description/meshes/visual/base_link.stl"/>
         </geometry>
+        <material name = "light_grey"/>
       </visual>
       <collision>
@@ -33,4 +36,5 @@
           <mesh filename="package://abb_irb120_description/meshes/visual/link_1.stl"/>
         </geometry>
+        <material name = "light_grey"/>
       </visual>
       <collision>
@@ -52,4 +56,5 @@
           <mesh filename="package://abb_irb120_description/meshes/visual/link_2.stl"/>
         </geometry>
+        <material name = "light_grey"/>
       </visual>
       <collision>
@@ -71,4 +76,5 @@
           <mesh filename="package://abb_irb120_description/meshes/visual/link_3.stl"/>
         </geometry>
+        <material name = "light_grey"/>
       </visual>
       <collision>
@@ -90,4 +96,5 @@
           <mesh filename="package://abb_irb120_description/meshes/visual/link_4.stl"/>
         </geometry>
+        <material name = "light_grey"/>
       </visual>
       <collision>
@@ -109,4 +116,5 @@
           <mesh filename="package://abb_irb120_description/meshes/visual/link_5.stl"/>
         </geometry>
+        <material name = "light_grey"/>
       </visual>
       <collision>
@@ -128,4 +136,5 @@
           <mesh filename="package://abb_irb120_description/meshes/visual/link_6.stl"/>
         </geometry>
+        <material name = "light_grey"/>
       </visual>
       <collision>
@@ -142,5 +151,5 @@
       <parent link="${prefix}base_link"/>
       <child link="${prefix}link_1"/>
-      <limit effort="100.0" lower="-2.87979" upper="2.87979" velocity="4.36332"/>
+      <limit effort="1000.0" lower="-2.87979" upper="2.87979" velocity="4.36332"/>
       <axis xyz="0 0 1"/>
       <dynamics damping="0.0" friction="0.0"/>
@@ -215,4 +224,5 @@
           <mesh filename="package://abb_irb120_description/meshes/visual/herramienta.stl"/>
         </geometry>
+        <material name = "grey"/>
       </visual>
       <collision>

File: abb_irb120_description/urdf/irb120_gazebo.xacro (robot description, xacro)
@@ -26,28 +26,4 @@
     <gazebo reference="link_5"><self_collide>false</self_collide></gazebo>
     <gazebo reference="link_6"><self_collide>false</self_collide></gazebo>
-    <gazebo reference="base_link">
-      <material>Gazebo/Red</material>
-    </gazebo>
-    <gazebo reference="link_1">
-      <material>Gazebo/Red</material>
-    </gazebo>
-    <gazebo reference="link_2">
-      <material>Gazebo/Red</material>
-    </gazebo>
-    <gazebo reference="link_3">
-      <material>Gazebo/Red</material>
-    </gazebo>
-    <gazebo reference="link_4">
-      <material>Gazebo/Red</material>
-    </gazebo>
-    <gazebo reference="link_5">
-      <material>Gazebo/Red</material>
-    </gazebo>
-    <gazebo reference="link_6">
-      <material>Gazebo/Black</material>
-    </gazebo>
-    <gazebo reference="herramienta_link">
-      <material>Gazebo/Grey</material>
-    </gazebo>
   </xacro:macro>
 </robot>

Commit message: Union del rover con el ABB

File: abb_irb120_description/urdf/irb120_3_58_macro.xacro (robot description, xacro)
@@ -240,13 +240,7 @@
   </xacro:macro>
   <xacro:abb_irb120_3_58 prefix="" />
-    <link name="world" />
-    <joint name="world_to_base" type="fixed">
-        <parent link="world" />
-        <child link="base_link" />
-        <origin xyz="0 0 0" rpy="0 0 0" />
-    </joint>
-    <xacro:include filename="irb120_gazebo.xacro" />
-    <xacro:include filename="irb120_control.xacro" />
-    <xacro:irb120_gazebo_plugins />
-    <xacro:irb120_ros2_control />
+  <xacro:include filename="irb120_gazebo.xacro" />
+  <xacro:include filename="irb120_control.xacro" />
+  <xacro:irb120_gazebo_plugins />
+  <xacro:irb120_ros2_control />
 </robot>

File: abb_irb120_description/urdf/irb120_gazebo.xacro (robot description, xacro)
@@ -2,10 +2,15 @@
 <robot xmlns:xacro="http://www.ros.org/wiki/xacro">
   <xacro:macro name="irb120_gazebo_plugins" params="">
+    <!--plugin de ros2 control para mover el brazo en gazebo-->
     <gazebo>
       <plugin filename="gz_ros2_control-system"
               name="gz_ros2_control::GazeboSimROS2ControlPlugin">
-        <parameters>$(find abb_irb120_description)/config/controllers.yaml</parameters>
+        <parameters>$(find multi_robot_bringup)/config/controllers.yaml</parameters>
+        <ros>
+          <remapping>/robot_description:=/rover/robot_description</remapping>
+        </ros>
       </plugin>
     </gazebo>
+    <!--publicar joint states-->
     <gazebo>
       <plugin filename="gz-sim-joint-state-publisher-system"
@@ -19,4 +24,5 @@
       </plugin>
     </gazebo>
+    <!--desactiva las colisiones internas del brazo-->
     <gazebo reference="base_link"><self_collide>false</self_collide></gazebo>
     <gazebo reference="link_1"><self_collide>false</self_collide></gazebo>

File: rover_description/urdf/rover.xacro (robot description, xacro)
@@ -50,8 +50,8 @@
     </collision>
     <inertial>
-      <mass value="5.0"/>
-      <inertia ixx="0.1" ixy="0.0" ixz="0.0"
-               iyy="0.1" iyz="0.0"
-               izz="0.1"/>
+      <mass value="50.0"/>
+      <inertia ixx="1.0" ixy="0.0" ixz="0.0"
+               iyy="1.0" iyz="0.0"
+               izz="1.0"/>
     </inertial>
   </link>

Commit message: Arreglado conflicto de nombres

File: abb_irb120_description/urdf/irb120_3_58_macro.xacro (robot description, xacro)
@@ -1,4 +1,4 @@
 <?xml version="1.0"?>
-<robot name="irb120_3_58" xmlns:xacro="http://www.ros.org/wiki/xacro">
+<robot xmlns:xacro="http://www.ros.org/wiki/xacro">
   <material name="light_grey"><color rgba="0.9 0.9 0.9 1"/></material>
   <material name="grey"><color rgba="0.4 0.4 0.4 1"/></material>
@@ -239,8 +239,3 @@
     </joint>
   </xacro:macro>
-  <xacro:abb_irb120_3_58 prefix="" />
-  <xacro:include filename="irb120_gazebo.xacro" />
-  <xacro:include filename="irb120_control.xacro" />
-  <xacro:irb120_gazebo_plugins />
-  <xacro:irb120_ros2_control />
 </robot>

File: abb_irb120_description/urdf/irb120_control.xacro (robot description, xacro)
@@ -19,10 +19,10 @@
       </xacro:macro>
       <!-- Llamadas a los joints -->
-      <xacro:arm_joint name="joint_1" lower="-2.879" upper="2.879"/>
-      <xacro:arm_joint name="joint_2" lower="-1.919" upper="1.919"/>
-      <xacro:arm_joint name="joint_3" lower="-1.919" upper="1.221"/>
-      <xacro:arm_joint name="joint_4" lower="-2.792" upper="2.792"/>
-      <xacro:arm_joint name="joint_5" lower="-2.094" upper="2.094"/>
-      <xacro:arm_joint name="joint_6" lower="-6.981" upper="6.981"/>
+      <xacro:arm_joint name="arm_joint_1" lower="-2.879" upper="2.879"/>
+      <xacro:arm_joint name="arm_joint_2" lower="-1.919" upper="1.919"/>
+      <xacro:arm_joint name="arm_joint_3" lower="-1.919" upper="1.221"/>
+      <xacro:arm_joint name="arm_joint_4" lower="-2.792" upper="2.792"/>
+      <xacro:arm_joint name="arm_joint_5" lower="-2.094" upper="2.094"/>
+      <xacro:arm_joint name="arm_joint_6" lower="-6.981" upper="6.981"/>
     </ros2_control>
   </xacro:macro>

File: abb_irb120_description/urdf/irb120_gazebo.xacro (robot description, xacro)
@@ -8,4 +8,5 @@
         <parameters>$(find multi_robot_bringup)/config/controllers.yaml</parameters>
         <ros>
+          <namespace>/rover</namespace>
           <remapping>/robot_description:=/rover/robot_description</remapping>
         </ros>
@@ -16,20 +17,20 @@
       <plugin filename="gz-sim-joint-state-publisher-system"
               name="gz::sim::systems::JointStatePublisher">
-        <joint_name>joint_1</joint_name>
-        <joint_name>joint_2</joint_name>
-        <joint_name>joint_3</joint_name>
-        <joint_name>joint_4</joint_name>
-        <joint_name>joint_5</joint_name>
-        <joint_name>joint_6</joint_name>
+        <joint_name>arm_joint_1</joint_name>
+        <joint_name>arm_joint_2</joint_name>
+        <joint_name>arm_joint_3</joint_name>
+        <joint_name>arm_joint_4</joint_name>
+        <joint_name>arm_joint_5</joint_name>
+        <joint_name>arm_joint_6</joint_name>
       </plugin>
     </gazebo>
     <!--desactiva las colisiones internas del brazo-->
-    <gazebo reference="base_link"><self_collide>false</self_collide></gazebo>
-    <gazebo reference="link_1"><self_collide>false</self_collide></gazebo>
-    <gazebo reference="link_2"><self_collide>false</self_collide></gazebo>
-    <gazebo reference="link_3"><self_collide>false</self_collide></gazebo>
-    <gazebo reference="link_4"><self_collide>false</self_collide></gazebo>
-    <gazebo reference="link_5"><self_collide>false</self_collide></gazebo>
-    <gazebo reference="link_6"><self_collide>false</self_collide></gazebo>
+    <gazebo reference="arm_base_link"><self_collide>false</self_collide></gazebo>
+    <gazebo reference="arm_link_1"><self_collide>false</self_collide></gazebo>
+    <gazebo reference="arm_link_2"><self_collide>false</self_collide></gazebo>
+    <gazebo reference="arm_link_3"><self_collide>false</self_collide></gazebo>
+    <gazebo reference="arm_link_4"><self_collide>false</self_collide></gazebo>
+    <gazebo reference="arm_link_5"><self_collide>false</self_collide></gazebo>
+    <gazebo reference="arm_link_6"><self_collide>false</self_collide></gazebo>
   </xacro:macro>
 </robot>

File: multi_robot_bringup/urdf/rover_abb.xacro (robot description, xacro)
@@ -2,17 +2,13 @@
 <robot name="rover_abb" xmlns:xacro="http://www.ros.org/wiki/xacro">
     <xacro:arg name="prefix" default="" />
-    <!--xacros del rover-->
-    <xacro:include filename="$(find rover_description)/urdf/rover.xacro"/>
-    <xacro:include filename="$(find rover_description)/urdf/gazebo_plugins.xacro"/>
-    <xacro:include filename="$(find rover_description)/urdf/lidar.xacro"/>
-    <!--xacro del ABB-->
-    <xacro:include filename="$(find abb_irb120_description)/urdf/irb120_3_58_macro.xacro" />
+    <!--xacro del rover-->
+    <xacro:include filename="$(find rover_description)/urdf/robot.urdf.xacro"/>
+    <!--xacros del ABB-->
+    <xacro:include filename="$(find abb_irb120_description)/urdf/abb.xacro" />
     <!--link para unir el rover con el abb-->
     <joint name="union_rover_abb" type="fixed">
         <parent link="$(arg prefix)base_link"/>
-        <child link="base_link"/>
+        <child link="arm_base_link"/>
         <origin xyz="0.2 0 0.352" rpy="0 0 0"/>
     </joint>
-    <!--lidar-->
-    <xacro:lidar_plugin prefix="$(arg prefix)"/>
 </robot>

Commit message: Tengo que arreglar que despues de mover el brazo el rover no toma nuevas metas

File: abb_irb120_description/urdf/irb120_3_58_macro.xacro (robot description, xacro)
@@ -159,5 +159,5 @@
       <parent link="${prefix}link_1"/>
       <child link="${prefix}link_2"/>
-      <limit effort="100.0" lower="-1.91986" upper="1.91986" velocity="4.36332"/>
+      <limit effort="1000.0" lower="-1.91986" upper="1.91986" velocity="4.36332"/>
       <axis xyz="0 1 0"/>
       <dynamics damping="0.0" friction="0.0"/>
@@ -167,5 +167,5 @@
       <parent link="${prefix}link_2"/>
       <child link="${prefix}link_3"/>
-      <limit effort="100.0" lower="-1.91986" upper="1.22173" velocity="4.36332"/>
+      <limit effort="1000.0" lower="-1.91986" upper="1.22173" velocity="4.36332"/>
       <axis xyz="0 1 0"/>
       <dynamics damping="0.0" friction="0.0"/>
@@ -175,5 +175,5 @@
       <parent link="${prefix}link_3"/>
       <child link="${prefix}link_4"/>
-      <limit effort="100.0" lower="-2.79253" upper="2.79253" velocity="5.58505"/>
+      <limit effort="1000.0" lower="-2.79253" upper="2.79253" velocity="5.58505"/>
       <axis xyz="1 0 0"/>
       <dynamics damping="0.0" friction="0.0"/>
@@ -183,5 +183,5 @@
       <parent link="${prefix}link_4"/>
       <child link="${prefix}link_5"/>
-      <limit effort="100.0" lower="-2.094395" upper="2.094395" velocity="5.58505"/>
+      <limit effort="1000.0" lower="-2.094395" upper="2.094395" velocity="5.58505"/>
       <axis xyz="0 1 0"/>
       <dynamics damping="0.0" friction="0.0"/>
@@ -191,5 +191,5 @@
       <parent link="${prefix}link_5"/>
       <child link="${prefix}link_6"/>
-      <limit effort="100.0" lower="-6.98132" upper="6.98132" velocity="7.33038"/>
+      <limit effort="1000.0" lower="-6.98132" upper="6.98132" velocity="7.33038"/>
       <axis xyz="1 0 0"/>
       <dynamics damping="0.0" friction="0.0"/>
